File: Hardware/Top/Watch-It-TOP.sch (EAGLE design)
At the start: 51 parts, among them SW1 SWITCH.MOM, SW2 SWITCH.MOM, U2 NRF52832_MODULE_MDBT42, U4 PCF8523

Commit message: routing
Parts:
- added C20, C6: 47p, LinnesLab-Passives:CAPACITOR0603
- added C5: 100n, LinnesLab-Passives:CAPACITOR0603
- added JP2: (no value), LinnesLab-Switches:JUMPER-SMT_2_NO_SILK
- added LED5: RED, LinnesLab-LED:LED0603
- added LED6: YELLOW, LinnesLab-LED:LED0603
- added R1, R2: 0, LinnesLab-Passives:RESISTOR0603
- added R12, R13: 27, LinnesLab-Passives:RESISTOR0603
- added R14, R15: 1k, LinnesLab-Passives:RESISTOR0603
- added U5: FT231XS, LinnesLab-DigitalIC:FT231XS
Connections:
- removed net RXD: U2.P0.08
- removed net TXD: U2.P0.06
- removed net VBATT: U4.VBAT
- new net !CTS: JP2.2, U5.!CTS
- new net FT3V3: U5.3V3OUT
- new net N$23: R12.2, U5.USBDM
- new net N$24: R13.2, U5.USBDP
- new net N$25: LED5.C, R14.2
- new net N$26: LED6.C, R15.2
- new net RXD.FT: U5.RXD
- new net RXD.NRF: R1.2, U2.P0.08
- new net RXDFT: R2.1
- new net RXLED: R14.1, U5.CBUS1
- new net TXD.FT: U5.TXD
- new net TXD.NRF: R2.2, U2.P0.06
- new net TXDFT: R1.1
- new net TXLED: R15.1, U5.CBUS2
- net 3.3V: now also C5.2, LED5.A, LED6.A, U5.!RESET, U5.VCCIO
- net DTR: now also U5.!DTR
- net GND: now also C20.1, C5.1, C6.2, JP2.1, U5.GND@16, U5.GND@6
- net SCL: now also R9.1; no longer R8.1
- net SDA: now also R8.1; no longer R9.1
- net USB+: now also C6.1, R13.1
- net USB-: now also C20.2, R12.1
- net V_USB: now also U5.VCC
Other:
- note added: "I don't remember if CTS needs to be grounded or left floating so here's a jumper to ground so it can be configued either way dynamically."
- note added: "TXD goes to RX on the other device RXD goes to TX on the other device"
- moved on the sheet: R8, R9

Commit message: made connections and added pins
Parts:
- added J1: (no value), LinnesLab-Connectors:CONN_07
Connections:
- removed net BATT: R18.1, R19.2
- removed net CHRG.STAT: CHRG3.STAT, R17.1
- new net A4/BATT: R18.1, R19.2, U2.P0.28/AIN4
- new net D27/CHRG.STATUS: CHRG3.STAT, R17.1, U2.P0.27
- new net D7/SD.CS: U2.P0.07
Other:
- note added: "Digital Output"
- note added: "FTDI Serial-to-USB Converter"
- note added: "Notes"
- moved on the sheet: C20, C5, C6, JP2, LED5, LED6, R1, R12, R13, R14, R15, R2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

Commit message: week 4 edits
Connections:
- removed net CS.OLED: U3./CS
- removed net DC.OLED: U3.DC/I2C_SA0
- removed net RESET.OLED: U3./RES
- removed net SW1: SW1.1, SW2.1
- new net A6/TIA: J1.5, U2.P0.30/AIN6
- new net A7/PPG: J1.7, U2.P0.31/AIN7
- new net D11/SW1: SW1.1, U2.P0.11
- new net D15/SW2: SW2.1, U2.P0.15
- new net D16/CS.OLED: U2.P0.16, U3./CS
- new net D29/LED.CTRL: J1.6, U2.P0.29/AIN5
- new net D3/RESET.OLED: U2.P0.03/AIN1, U3./RES
- new net D4/DC.OLED: U2.P0.04/AIN2, U3.DC/I2C_SA0
- new net D5/CD1: U2.P0.05/AIN3
Changed lines of the file:
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@@
 <text x="396.24" y="812.8" size="1.27" layer="97">100nF+10K @ 3.3V =
 ~1.2ms to 0.7VCC</text>
-<text x="154.94" y="855.98" size="1.27" layer="97">SPECIAL / PORT / PIN ON PACKAGE / GPIO(D_or_A) / Comments
+<text x="152.4" y="853.44" size="1.27" layer="97">SPECIAL / PORT / PIN ON PACKAGE / GPIO(D_or_A) / Comments
 SDA / P0.25 / pin2 / D25
 SCL / P0.26 / pin3 / D26
@@
 <net name="N$6" class="0">
 <segment>
-<wire x1="248.92" y1="810.26" x2="248.92" y2="807.72" width="0.1524" layer="91"/>
 <wire x1="243.84" y1="830.58" x2="243.84" y2="815.34" width="0.1524" layer="91"/>
-<wire x1="243.84" y1="815.34" x2="248.92" y2="815.34" width="0.1524" layer="91"/>
-<wire x1="248.92" y1="815.34" x2="248.92" y2="810.26" width="0.1524" layer="91"/>
-<junction x="248.92" y="810.26"/>
+<wire x1="243.84" y1="815.34" x2="246.38" y2="815.34" width="0.1524" layer="91"/>
+<wire x1="246.38" y1="815.34" x2="246.38" y2="810.26" width="0.1524" layer="91"/>
+<pinref part="XTAL2" gate="G$1" pin="2"/>
+<wire x1="246.38" y1="810.26" x2="243.84" y2="810.26" width="0.1524" layer="91"/>
+<pinref part="U2" gate="G$1" pin="P0.01/XL2"/>
 <pinref part="C9" gate="G$1" pin="1"/>
-<pinref part="XTAL2" gate="G$1" pin="2"/>
-<wire x1="248.92" y1="810.26" x2="243.84" y2="810.26" width="0.1524" layer="91"/>
-<pinref part="U2" gate="G$1" pin="P0.01/XL2"/>
+<wire x1="248.92" y1="807.72" x2="248.92" y2="810.26" width="0.1524" layer="91"/>
+<wire x1="248.92" y1="810.26" x2="246.38" y2="810.26" width="0.1524" layer="91"/>
+<junction x="246.38" y="810.26"/>
 </segment>
 </net>
@@
 </segment>
 <segment>
-<label x="480.06" y="822.96" size="1.778" layer="95"/>
 <pinref part="U3" gate="G$1" pin="D0/SPI_SCLK/I2C_SCK"/>
-<wire x1="505.46" y1="822.96" x2="480.06" y2="822.96" width="0.1524" layer="91"/>
+<wire x1="505.46" y1="822.96" x2="500.38" y2="822.96" width="0.1524" layer="91"/>
+<label x="500.38" y="822.96" size="1.27" layer="95" rot="R180" xref="yes"/>
 </segment>
 <segment>
@@
 </segment>
 <segment>
-<label x="480.06" y="820.42" size="1.778" layer="95"/>
 <pinref part="U3" gate="G$1" pin="D1/SPI_SDIN/I2C_SDA"/>
-<wire x1="505.46" y1="820.42" x2="480.06" y2="820.42" width="0.1524" layer="91"/>
+<wire x1="505.46" y1="820.42" x2="500.38" y2="820.42" width="0.1524" layer="91"/>
+<label x="500.38" y="820.42" size="1.27" layer="95" rot="R180" xref="yes"/>
 </segment>
 <segment>
@@
 </segment>
 </net>
-<net name="DC.OLED" class="0">
-<segment>
-<label x="480.06" y="830.58" size="1.778" layer="95"/>
-<pinref part="U3" gate="G$1" pin="DC/I2C_SA0"/>
-<wire x1="505.46" y1="830.58" x2="480.06" y2="830.58" width="0.1524" layer="91"/>
-</segment>
-</net>
-<net name="RESET.OLED" class="0">
-<segment>
-<label x="480.06" y="833.12" size="1.778" layer="95"/>
-<pinref part="U3" gate="G$1" pin="/RES"/>
-<wire x1="505.46" y1="833.12" x2="480.06" y2="833.12" width="0.1524" layer="91"/>
-</segment>
-</net>
 <net name="N$1" class="0">
 <segment>
@@
 <pinref part="U3" gate="G$1" pin="VCOMH"/>
 <wire x1="505.46" y1="800.1" x2="487.68" y2="800.1" width="0.1524" layer="91"/>
-</segment>
-</net>
-<net name="CS.OLED" class="0">
-<segment>
-<label x="480.06" y="835.66" size="1.778" layer="95"/>
-<pinref part="U3" gate="G$1" pin="/CS"/>
-<wire x1="505.46" y1="835.66" x2="480.06" y2="835.66" width="0.1524" layer="91"/>
 </segment>
 </net>
@@
 </segment>
 </net>
-<net name="SW1" class="0">
-<segment>
-<pinref part="SW1" gate="G$1" pin="1"/>
-<wire x1="472.44" y1="736.6" x2="469.9" y2="736.6" width="0.1524" layer="91"/>
-<label x="469.9" y="736.6" size="1.27" layer="95" rot="R180" xref="yes"/>
-</segment>
-<segment>
-<pinref part="SW2" gate="G$1" pin="1"/>
-<wire x1="505.46" y1="736.6" x2="502.92" y2="736.6" width="0.1524" layer="91" style="longdash"/>
-<label x="502.92" y="736.6" size="1.27" layer="95" rot="R180" xref="yes"/>
-</segment>
-</net>
 <net name="N$23" class="0">
 <segment>
@@
 </segment>
 </net>
+<net name="D5/CD1" class="0">
+<segment>
+<pinref part="U2" gate="G$1" pin="P0.05/AIN3"/>
+<wire x1="254" y1="830.58" x2="254" y2="828.04" width="0.1524" layer="91"/>
+<label x="254" y="828.04" size="1.27" layer="95" rot="R270" xref="yes"/>
+</segment>
+</net>
+<net name="D11/SW1" class="0">
+<segment>
+<pinref part="U2" gate="G$1" pin="P0.11"/>
+<wire x1="276.86" y1="843.28" x2="279.4" y2="843.28" width="0.1524" layer="91"/>
+<label x="279.4" y="843.28" size="1.27" layer="95" xref="yes"/>
+</segment>
+<segment>
+<pinref part="SW1" gate="G$1" pin="1"/>
+<wire x1="472.44" y1="736.6" x2="469.9" y2="736.6" width="0.1524" layer="91"/>
+<label x="469.9" y="736.6" size="1.27" layer="95" rot="R180" xref="yes"/>
+</segment>
+</net>
+<net name="D15/SW2" class="0">
+<segment>
+<pinref part="U2" gate="G$1" pin="P0.15"/>
+<wire x1="276.86" y1="853.44" x2="279.4" y2="853.44" width="0.1524" layer="91"/>
+<label x="279.4" y="853.44" size="1.27" layer="95" xref="yes"/>
+</segment>
+<segment>
+<pinref part="SW2" gate="G$1" pin="1"/>
+<wire x1="505.46" y1="736.6" x2="502.92" y2="736.6" width="0.1524" layer="91" style="longdash"/>
+<label x="502.92" y="736.6" size="1.27" layer="95" rot="R180" xref="yes"/>
+</segment>
+</net>
+<net name="D16/CS.OLED" class="0">
+<segment>
+<pinref part="U2" gate="G$1" pin="P0.16"/>
+<wire x1="276.86" y1="855.98" x2="279.4" y2="855.98" width="0.1524" layer="91"/>
+<label x="279.4" y="855.98" size="1.27" layer="95" xref="yes"/>
+</segment>
+<segment>
+<pinref part="U3" gate="G$1" pin="/CS"/>
+<wire x1="505.46" y1="835.66" x2="500.38" y2="835.66" width="0.1524" layer="91"/>
+<label x="500.38" y="835.66" size="1.27" layer="95" rot="R180" xref="yes"/>
+</segment>
+</net>
+<net name="D4/DC.OLED" class="0">
+<segment>
+<pinref part="U2" gate="G$1" pin="P0.04/AIN2"/>
+<wire x1="251.46" y1="830.58" x2="251.46" y2="828.04" width="0.1524" layer="91"/>
+<label x="251.46" y="828.04" size="1.27" layer="95" rot="R270" xref="yes"/>
+</segment>
+<segment>
+<pinref part="U3" gate="G$1" pin="DC/I2C_SA0"/>
+<wire x1="505.46" y1="830.58" x2="500.38" y2="830.58" width="0.1524" layer="91"/>
+<label x="500.38" y="830.58" size="1.27" layer="95" rot="R180" xref="yes"/>
+</segment>
+</net>
+<net name="D3/RESET.OLED" class="0">
+<segment>
+<pinref part="U2" gate="G$1" pin="P0.03/AIN1"/>
+<wire x1="248.92" y1="830.58" x2="248.92" y2="828.04" width="0.1524" layer="91"/>
+<label x="248.92" y="828.04" size="1.27" layer="95" rot="R270" xref="yes"/>
+</segment>
+<segment>
+<pinref part="U3" gate="G$1" pin="/RES"/>
+<wire x1="505.46" y1="833.12" x2="500.38" y2="833.12" width="0.1524" layer="91"/>
+<label x="500.38" y="833.12" size="1.27" layer="95" rot="R180" xref="yes"/>
+</segment>
+</net>
+<net name="D29/LED.CTRL" class="0">
+<segment>
+<pinref part="U2" gate="G$1" pin="P0.29/AIN5"/>
+<wire x1="231.14" y1="858.52" x2="228.6" y2="858.52" width="0.1524" layer="91"/>
+<label x="228.6" y="858.52" size="1.27" layer="95" rot="R180" xref="yes"/>
+</segment>
+<segment>
+<pinref part="J1" gate="G$1" pin="6"/>
+<wire x1="477.52" y1="985.52" x2="480.06" y2="985.52" width="0.1524" layer="91"/>
+<label x="480.06" y="985.52" size="1.27" layer="95" xref="yes"/>
+</segment>
+</net>
+<net name="A6/TIA" class="0">
+<segment>
+<pinref part="U2" gate="G$1" pin="P0.30/AIN6"/>
+<wire x1="231.14" y1="855.98" x2="228.6" y2="855.98" width="0.1524" layer="91"/>
+<label x="228.6" y="855.98" size="1.27" layer="95" rot="R180" xref="yes"/>
+</segment>
+<segment>
+<pinref part="J1" gate="G$1" pin="5"/>
+<wire x1="477.52" y1="982.98" x2="480.06" y2="982.98" width="0.1524" layer="91"/>
+<label x="480.06" y="982.98" size="1.27" layer="95" xref="yes"/>
+</segment>
+</net>
+<net name="A7/PPG" class="0">
+<segment>
+<pinref part="U2" gate="G$1" pin="P0.31/AIN7"/>
+<wire x1="231.14" y1="853.44" x2="228.6" y2="853.44" width="0.1524" layer="91"/>
+<label x="228.6" y="853.44" size="1.27" layer="95" rot="R180" xref="yes"/>
+</segment>
+<segment>
+<pinref part="J1" gate="G$1" pin="7"/>
+<wire x1="477.52" y1="988.06" x2="480.06" y2="988.06" width="0.1524" layer="91"/>
+<label x="480.06" y="988.06" size="1.27" layer="95" xref="yes"/>
+</segment>
+</net>
