File: Hardware/Top/Watch-It-TOP.brd (EAGLE design)
At the start: 38 x 38 mm, 51 parts, among them SW1 SWITCH.MOM, SW2 SWITCH.MOM, U2 NRF52832_MODULE_MDBT42, U4 PCF8523

Commit message: did some routing
Parts:
- moved R7 17.6 mm to (22.8, 15.9)
- moved R6 9.20 mm to (15.0, 15.4)
- moved C18 7.82 mm to (18.8, 23.0), turned to 270 degrees
- moved C16 7.77 mm to (20.2, 24.1)
- moved C7 6.46 mm to (17.6, 25.1)
- moved C19 4.26 mm to (10.9, 21.3)
- moved C13 4.01 mm to (8.23, 21.5), turned to 180 degrees
- moved C17 3.68 mm to (13.1, 21.7)
- moved R9 3.44 mm to (11.2, 25.2), turned to 0 degrees
- moved U3 3.35 mm to (17.6, 19.5)
- moved C15 2.44 mm to (9.53, 23.4), turned to 180 degrees
- moved XTAL3 2.35 mm to (1.68, 28.3)
- moved U4 2.02 mm to (5.94, 27.1)
- moved XTAL2 1.87 mm to (29.6, 18.3)
- moved C8 1.86 mm to (27.7, 15.6)
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Routing:
- net GND: track 0.00 -> 39.1 mm, vias 0 -> 13
- net SDA: track 0.00 -> 22.7 mm, vias 0 -> 2
- net MOSI: track 0.00 -> 19.8 mm, vias 0 -> 1
- net 3.3V: track 0.00 -> 19.2 mm, vias 0 -> 4
- net SCL: track 0.00 -> 19.1 mm
- net SCK: track 0.00 -> 17.2 mm, vias 0 -> 1
- net N$13: track 0.00 -> 10.4 mm
- net N$12: track 0.00 -> 9.90 mm
- net N$15: track 0.00 -> 9.17 mm
- net N$6: track 0.00 -> 6.26 mm
- net N$4: track 0.00 -> 5.91 mm
- net N$7: track 0.00 -> 5.29 mm
- net N$8: track 0.00 -> 5.10 mm
- net N$11: track 0.00 -> 5.05 mm
- net N$2: track 0.00 -> 4.44 mm
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- added copper zone on layer 1, net 9V
- added copper zone on layer 16, net GND\

Commit message: routing
Parts:
- added C20, C6: 47p, LinnesLab-Passives:C0603
- added C5: 100n, LinnesLab-Passives:C0603
- added JP2: (no value), LinnesLab-Switches:SMT-JUMPER_2_NO_SILK
- added LED5: RED, LinnesLab-LED:LED-0603
- added LED6: YELLOW, LinnesLab-LED:LED-0603
- added R1, R2: 0, LinnesLab-Passives:R0603
- added R12, R13: 27, LinnesLab-Passives:R0603
- added R14, R15: 1k, LinnesLab-Passives:R0603
- added U5: FT231XS, LinnesLab-DigitalIC:SSOP20_L
- moved R9 39.6 mm to (0.53, -12.9)
- moved R8 39.5 mm to (0.53, -10.2), turned to 0 degrees
Connections:
- net VBATT renamed VBAT
- removed net RXD: U2.21
- removed net TXD: U2.19
- new net !CTS: JP2.2, U5.9
- new net FT3V3: U5.13
- new net N$23: R12.2, U5.12
- new net N$24: R13.2, U5.11
- new net N$25: LED5.C, R14.2
- new net N$26: LED6.C, R15.2
- new net RXD.FT: U5.4
- new net RXD.NRF: R1.2, U2.21
- new net RXDFT: R2.1
- new net RXLED: R14.1, U5.17
- new net TXD.FT: U5.20
- new net TXD.NRF: R2.2, U2.19
- new net TXDFT: R1.1
- new net TXLED: R15.1, U5.10
- net 3.3V: now also C5.2, LED5.A, LED6.A, U5.14, U5.3
- net DTR: now also U5.1
- net GND: now also C20.1, C5.1, C6.2, JP2.1, U5.16, U5.6
- net SCL: now also R9.1; no longer R8.1
- net SDA: now also R8.1; no longer R9.1
- net USB+: now also C6.1, R13.1
- net USB-: now also C20.2, R12.1
- net V_USB: now also U5.15
Routing:
- net SCL: track 19.1 -> 16.4 mm
- net 3.3V: track 19.2 -> 17.6 mm, vias 4 -> 3
- net SDA: track 22.7 -> 21.7 mm

Commit message: made connections and added pins
Parts:
- added J1: (no value), LinnesLab-Connectors:1X07
- moved U5 6.14 mm to (14.9, 27.2)
- moved C7 2.54 mm to (18.9, 27.2)
- moved C2 0.54 mm to (7.98, 30.6)
- moved C17 0.26 mm to (13.1, 21.5)
Connections:
- removed net BATT: R18.1, R19.2
- removed net CHRG.STAT: CHRG3.1, R17.1
- new net A4/BATT: R18.1, R19.2, U2.5
- new net D27/CHRG.STATUS: CHRG3.1, R17.1, U2.4
- new net D7/SD.CS: U2.20
Routing:
- net SCL: track 16.4 -> 19.4 mm, vias 0 -> 2
- net 3.3V: track 17.6 -> 17.0 mm
- net SDA: track 21.7 -> 21.2 mm

Commit message: Almost done routing
Parts:
- moved LED6 70.2 mm to (2.79, 19.8)
- moved C6 70.1 mm to (6.27, 8.10), turned to 90 degrees
- moved C20 69.5 mm to (6.83, 3.28)
- moved R15 65.7 mm to (4.72, 18.3), turned to 180 degrees
- moved R12 59.1 mm to (5.69, 13.2)
- moved C5 57.6 mm to (11.2, 27.9), turned to 90 degrees
- moved JP2 48.6 mm to (5.46, 23.1)
- moved C14 48.5 mm to (3.00, 31.8), turned to 90 degrees
- moved D1 47.6 mm to (1.45, 32.0), turned to 270 degrees
- moved LED5 47.4 mm to (23.3, 33.6)
- moved R5 46.1 mm to (1.57, 35.1)
- moved R14 45.6 mm to (22.8, 30.8)
- moved R13 43.2 mm to (17.8, 21.1), turned to 90 degrees
- moved R9 42.9 mm to (9.63, 29.1), turned to 90 degrees
- moved R2 39.4 mm to (31.9, 17.9), turned to 90 degrees
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Connections:
- removed net CS.OLED: U3.13
- removed net DC.OLED: U3.15
- removed net RESET.OLED: U3.14
- removed net SW1: SW1.A1, SW2.A1
- new net A6/TIA: J1.5, U2.7
- new net A7/PPG: J1.7, U2.8
- new net D11/SW1: SW1.A1, U2.25
- new net D15/SW2: SW2.A1, U2.29
- new net D16/CS.OLED: U2.30, U3.13
- new net D29/LED.CTRL: J1.6, U2.6
- new net D3/RESET.OLED: U2.16, U3.14
- new net D4/DC.OLED: U2.17, U3.15
- new net D5/CD1: U2.18
Routing:
- net GND: track 39.2 -> 99.8 mm, vias 13 -> 23
- net D15/SW2: track 0.00 -> 37.7 mm, vias 0 -> 2
- net D11/SW1: track 0.00 -> 36.2 mm, vias 0 -> 2
- net D27/CHRG.STATUS: track 0.00 -> 33.7 mm, vias 0 -> 2
- net USB+: track 0.00 -> 25.7 mm, vias 0 -> 2
- net VIN: track 0.00 -> 24.0 mm
- net VLIPO: track 0.00 -> 19.4 mm
- net D4/DC.OLED: track 0.00 -> 19.3 mm, vias 0 -> 2
- net V_USB: track 0.00 -> 14.8 mm, vias 0 -> 1
- net A7/PPG: track 0.00 -> 14.7 mm, vias 0 -> 1
- net A6/TIA: track 0.00 -> 14.4 mm
- net USB-: track 0.00 -> 13.8 mm, vias 0 -> 1
- net 3.3V: track 17.0 -> 29.2 mm, vias 3 -> 9
- net D29/LED.CTRL: track 0.00 -> 11.6 mm
- net TXLED: track 0.00 -> 11.3 mm, vias 0 -> 2
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
Commit message: finished routing
Parts:
- moved LED4 22.4 mm to (26.0, 13.0), turned to 180 degrees
- moved LED3 22.0 mm to (25.9, 11.0), turned to 180 degrees
- moved R4 17.8 mm to (29.5, 12.7), turned to 0 degrees
- moved R3 17.1 mm to (29.5, 11.1), turned to 0 degrees
- moved C11 3.49 mm to (35.0, 14.1)
- moved C10 1.42 mm to (35.1, 18.3)
- moved CORTEX1 0.91 mm to (21.1, 35.5)
- moved U2 0.73 mm to (30.5, 28.8)
- moved LED5 0.71 mm to (23.1, 32.9), turned to 180 degrees
- moved C19 0.54 mm to (11.5, 21.2)
- moved R5 0.46 mm to (2.01, 35.3)
- moved C14 0.41 mm to (3.02, 31.3)
- moved XTAL2 0.39 mm to (29.2, 18.4)
- moved R1 0.36 mm to (33.4, 17.8)
- moved C16 0.33 mm to (20.3, 22.9)
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Routing:
- net GND: track 99.8 -> 144.5 mm, vias 23 -> 30
- net RESET: track 6.88 -> 47.3 mm, vias 0 -> 2
- net D16/CS.OLED: track 0.00 -> 26.0 mm, vias 0 -> 2
- net LED2: track 0.00 -> 24.6 mm, vias 0 -> 2
- net A4/BATT: track 0.00 -> 24.3 mm, vias 0 -> 2
- net LED1: track 0.00 -> 21.5 mm
- net 3.3V: track 29.2 -> 50.4 mm, vias 9 -> 7
- net DFU: track 0.00 -> 19.4 mm, vias 0 -> 1
- net D3/RESET.OLED: track 0.00 -> 19.3 mm, vias 0 -> 2
- net SWCLK: track 0.00 -> 18.4 mm, vias 0 -> 1
- net N$23: track 0.00 -> 17.8 mm, vias 0 -> 2
- net SCK: track 17.2 -> 34.9 mm, vias 1 -> 2
- net SWO: track 0.00 -> 17.6 mm, vias 0 -> 1
- net MOSI: track 19.8 -> 37.4 mm, vias 1 -> 2
- net SWDIO: track 0.00 -> 16.7 mm, vias 0 -> 1
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- added copper zone on layer 1, net 3.3V
- added copper zone on layer 16, net GND
- removed copper zone on layer 1, net 9V
- removed copper zone on layer 16, net GND\

Commit message: cleaned it up a bit
Routing:
- net 3.3V: track 50.4 -> 49.6 mm
- net SWDIO: track 16.7 -> 17.5 mm
Changed lines of the file:
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@@
 <wire x1="26.4414" y1="31.4074375" x2="26.4414" y2="31.2674" width="0.1524" layer="16"/>
 <wire x1="24.9792" y1="32.8696375" x2="26.4414" y2="31.4074375" width="0.1524" layer="16"/>
-<wire x1="26.4414" y1="31.2674" x2="26.9494" y2="30.7594" width="0.1524" layer="16"/>
-<wire x1="26.9494" y1="30.7594" x2="36.6058" y2="30.7594" width="0.1524" layer="16"/>
+<wire x1="26.4414" y1="31.2674" x2="27.8384" y2="29.8704" width="0.1524" layer="16"/>
+<wire x1="35.7168" y1="29.8704" x2="36.6058" y2="30.7594" width="0.1524" layer="16"/>
+<wire x1="35.7168" y1="29.8704" x2="27.8384" y2="29.8704" width="0.1524" layer="16"/>
 <via x="36.6058" y="30.7594" extent="1-16" drill="0.35"/>
 <wire x1="36.6058" y1="30.7594" x2="36.3772" y2="30.988" width="0.1524" layer="1"/>
@@
 <via x="12.0396" y="4.5466" extent="1-16" drill="0.35"/>
 <wire x1="12.0396" y1="4.5466" x2="11.94325" y2="4.45025" width="0.1524" layer="1"/>
-<wire x1="11.94325" y1="4.45025" x2="11.11995" y2="4.45025" width="0.1524" layer="1"/>
 </signal>
 <signal name="P0.09/NFC1">
