File: Hardware/Bottom/Watch-It-BOTTOM+.brd (EAGLE design)
At the start: 33 x 33 mm, 32 parts, among them U1 AD5242-SO16

Commit message: more routing
Parts:
- added C63, C64, C76, C78, C79, C80, C81, C82, C87: 100n, LinnesLab-Passives:C0603
- added C65, C70, C71, C77, C83: 1u, LinnesLab-Passives:C0603
- added C66, C67, C74, C75: 33p, LinnesLab-Passives:C0603
- added C68, C69: 10n, LinnesLab-Passives:C0603
- added C72, C73, C84, C85, C86: 10u, LinnesLab-Passives:C0603.POLAR
- added J6: AVR_SPI_PROG_3X2NS, LinnesLab-Connectors:2X3-NS
- added J7: (no value), LinnesLab-Connectors:AUDIO_JACK_3.5MM_TRRS_SMD_RA
- added R2: 10k, LinnesLab-Passives:R0805
- added R48, R49, R50, R61, R64: 10k, LinnesLab-Passives:R0603
- added R51, R52, R53, R57, R58, R59, R60: 100k, LinnesLab-Passives:R0603
- added R54: 1M, LinnesLab-Passives:R0603
- added R55, R62: 20, LinnesLab-Passives:R0603
- added R56, R63: 470, LinnesLab-Passives:R0603
- added THERM2: 10k, LinnesLab-Sensors:R0603
- added U10: VS1053B, LinnesLab-DigitalIC:LQFP-48
- added U8: (no value), LinnesLab-Power:SOT23-6
- added U9: ATMEGA328P_TQFP, LinnesLab-Microcontrollers:TQFP32-08
- added XTAL5: 12.288MHz, LinnesLab-Clocks:4-SMD.NOLEAD
- added XTAL6: 8MHz, LinnesLab-Clocks:4-SMD.NOLEAD.3.25MM-2.5MM
- moved Q1 4.19 mm to (16.4, 11.4)
- moved R16 3.61 mm to (13.0, 10.1)
- moved C18 2.96 mm to (17.5, 7.87)
- moved U1 2.79 mm to (24.4, 9.68)
- moved U$4 1.81 mm to (13.6, 6.73)
- moved R24 1.70 mm to (31.7, 19.4)
- moved C21 1.70 mm to (32.2, 13.3)
- moved R17 0.36 mm to (30.8, 28.1)
- moved R18 0.23 mm to (33.1, 28.3)
- moved R22 0.10 mm to (30.0, 22.9)
- moved R21 0.08 mm to (30.6, 25.9)
Connections:
- new net 1.8V: C71.1, C82.2, C83.2, C86.A, U10.24, U10.31, U10.5, U10.7, U8.1
- new net A0: U9.23
- new net A1: U9.24
- new net A2: U9.25
- new net A3: U9.26
- new net A6: U9.19
- new net A7: U9.22
- new net D5: U9.9
- new net DTR: C64.1
- new net GBUF: U10.42
- new net GPIO2: R58.2, U10.33
- new net LEFT: R55.2, R56.2, U10.46
- new net MIDI-RX: R60.1, U10.26, U9.1
- new net MP3-CS: U10.23, U9.10
- new net MP3-DCS: U10.13, U9.11
- new net MP3-DREQ: U10.8, U9.32
- new net MP3-EN1: U8.4
- new net MP3-EN2: U8.3
- new net MP3-GPIO1: R57.2, U10.34, U9.2
- new net MP3-MISO: J6.1, U10.30, U9.16
- new net MP3-MOSI: J6.4, U10.29, U9.15
- new net MP3-RST: R59.2
- new net MP3-RST-ATMEGA: C64.2, J6.5, R48.1, U9.29
- new net MP3-RST-VS: U10.3, U9.12
- new net MP3-RXD: U9.30
- new net MP3-SCK: J6.3, U10.28, U9.17
- new net MP3-SD: U9.13
- new net MP3-TXD: U9.31
- new net N$39: C63.2, U9.20
- new net N$40: U9.14
- new net N$41: C66.2, R54.2, U10.18, XTAL5.XTAL1
- new net N$42: C67.1, R54.1, U10.17, XTAL5.XTAL2
- new net N$43: R51.2, U10.10, U10.11, U10.12, U10.9
- new net N$44: R52.2, U10.25
- new net N$45: R53.2, U10.36
- new net N$46: C65.1, U10.44
- new net N$47: C68.2, R55.1
- new net N$48: C72.A, R56.1
- new net N$49: C69.2, R62.1
- new net N$50: C73.A, R63.1
- new net N$51: C74.2, U9.7, XTAL6.XTAL1
- new net N$52: C75.1, U9.8, XTAL6.XTAL2
- new net RIGHT: R62.2, R63.2, U10.39
- new net SPK-L: C72.C, J7.LEFT, R61.2
- new net SPK-R: C73.C, J7.RIGHT, R64.2
- new net THERM: R2.1, THERM2.1
- new net VIN: U8.5
- net 3.3V: now also C70.1, C76.2, C77.2, C78.2, C79.2, C80.2, C81.2, C84.A, C85.A, C87.2, J6.2, R2.2, R48.2, R49.2, R50.2, R60.2, U10.14, U10.19, U10.32, U10.38, U10.43, U10.45, U10.6, U8.6, U9.18, U9.4, U9.6
- net GND: now also C63.1, C65.2, C66.1, C67.2, C68.1, C69.1, C70.2, C71.2, C74.1, C75.2, C76.1, C77.1, C78.1, C79.1, C80.1, C81.1, C82.1, C83.1, C84.C, C85.C, C86.C, C87.1, J6.6, J7.GND, J7.GND/MIC, R51.1, R52.1, R53.1, R57.1, R58.1, R59.1, R61.1, R64.1, THERM2.2, U10.16, U10.20, U10.21, U10.22, U10.35, U10.37, U10.4, U10.40, U10.41, U10.47, U8.2, U9.21, U9.3, U9.5
- net SCL: now also R50.1, U9.28
- net SDA: now also R49.1, U9.27
Routing:
- net MP3-RST-ATMEGA: track 0.00 -> 39.1 mm, vias 0 -> 2
- net 3.3V: track 1.03 -> 39.9 mm, vias 0 -> 17
- net MP3-SCK: track 0.00 -> 35.7 mm, vias 0 -> 1
- net MP3-GPIO1: track 0.00 -> 33.4 mm, vias 0 -> 2
- net MP3-MISO: track 0.00 -> 31.4 mm
- net SCL: track 15.1 -> 33.5 mm, vias 2 -> 3
- net MP3-DREQ: track 0.00 -> 17.9 mm, vias 0 -> 2
- net RIGHT: track 0.00 -> 16.7 mm
- net SDA: track 16.7 -> 32.1 mm, vias 2 -> 3
- net LEFT: track 0.00 -> 12.0 mm
- net N$42: track 0.00 -> 11.4 mm
- net G.W2: track 29.4 -> 37.8 mm
- net 1.8V: track 0.00 -> 8.16 mm
- net N$41: track 0.00 -> 8.06 mm
- net GND: track 42.2 -> 34.9 mm
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